File: CPU_MEM-1.kicad_sch (KiCad schematic)
At the start: 23 parts, among them U8 S02, X4 SolderJumper_2_Open, X5 SolderJumper_2_Bridged

Commit message: add change apple2e
Parts:
- RP1: footprint Resistor_THT:R_Array_SIP10 -> Resistor_THT:R_Array_SIP9
- UB8, UE1: footprint (none) -> Package_DIP:DIP-14_W7.62mm_Socket_LongPads
- UE10: footprint (none) -> Package_DIP:DIP-28_W15.24mm_Socket_LongPads
- UE8: value 2365/2764 -> 2764; footprint (none) -> Package_DIP:DIP-28_W15.24mm_Socket_LongPads
- X4: footprint (none) -> Jumper:SolderJumper-2_P1.3mm_Open_RoundedPad1.0x1.5mm
- X5: footprint (none) -> Jumper:SolderJumper-2_P1.3mm_Bridged_RoundedPad1.0x1.5mm
- renumbered U8 to UB8
Connections:
- net +5V: now also UB1.20 (VCC), UB3.20 (VCC)
- net GND: now also UB1.10 (GND), UB3.10 (GND)
Other:
- note removed: "UB1 and UB3: no power pins"

Commit message: add change apple2e-3
Other:
- note removed: "JL: Setting MMU /PRAS to Input because it may be generated from PAL/HAL"
Changed lines of the file:
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@@
 		(title "CPU/MEM A2E NTSC")
-	)
-	(text "JL: Setting MMU /PRAS to Input because it may be generated from PAL/HAL"
-		(exclude_from_sim no)
-		(at 137.795 86.995 0)
-		(effects
-			(font
-				(size 1.27 1.27)
-			)
-			(justify left bottom)
-		)
 	)
 	(text "CD ROM"
