File: IO-2.kicad_sch (KiCad schematic)
At the start: 46 parts, among them J18 Conn_01x02, J19 Conn_01x02, J9 CASSETTE IN, Q5 MPSA13, X1 SolderJumper_2_Open, X2 SolderJumper_2_Bridged, X6 SolderJumper_2_Open

Commit message: add change apple2e
Parts:
- J19: footprint (none) -> Connector_PinHeader_1.00mm:PinHeader_1x02_P1.00mm_Vertical_SMD_Pin1Right
- J9: value CASSETTE IN -> AUDIO IN; footprint (none) -> Connector_Audio:Jack_3.5mm_CUI_SJ1-3525N_Horizontal; symbol Connector:Conn_Coaxial -> Connector_Audio:AudioJack3_Ground
- Q5: footprint (none) -> Package_TO_SOT_THT:TO-92_Inline
- RP1: footprint Resistor_THT:R_Array_SIP10 -> Resistor_THT:R_Array_SIP9
- SA1: footprint (none) -> Ferrite_THT:LairdTech_28C0236-0JW-10
- UA11: value MM741 -> LM741; footprint (none) -> Package_DIP:DIP-6_W7.62mm_Socket_LongPads
- UB2: footprint (none) -> Package_DIP:DIP-20_W7.62mm_LongPads
- UB5: footprint (none) -> Package_DIP:DIP-16_W7.62mm_Socket_LongPads
- UB8, UC5: footprint (none) -> Package_DIP:DIP-14_W7.62mm_Socket_LongPads
- UC10: footprint (none) -> Package_DIP:DIP-24_W7.62mm_Socket_LongPads
- UC12: footprint Package_DIP:CERDIP-20_W7.62mm_SideBrazed_LongPads_Socket -> Package_DIP:DIP-16_W7.62mm_Socket_LongPads
- UE14: footprint (none) -> Package_DIP:DIP-40_W15.24mm_Socket_LongPads
- X2, X6: footprint (none) -> Jumper:SolderJumper-2_P1.3mm_Open_RoundedPad1.0x1.5mm
Connections:
- net +5V: now also UB2.20 (VCC), UB5.16 (VCC), UC10.24 (VCC), UC12.16 (VCC)
- net GND: now also J9.G, UB2.10 (GND), UB5.8 (GND), UC10.12 (GND), UC12.8 (GND); no longer J9.2 (Ext)
- net at C11.2: now also J9.T; no longer J9.1 (In)
- no-connect marks 2 -> 4

Commit message: add change apple2e-2
Parts:
- C11, C34, C35, C37, C40, C71, C79, C80: footprint (none) -> Capacitor_THT:C_Axial_L3.8mm_D2.6mm_P10.00mm_Horizontal
- C36: footprint (none) -> OldComp:Cap_Cer_762
- C70: footprint (none) -> Capacitor_THT:C_Disc_D5.0mm_W2.5mm_P2.50mm
- J18: footprint (none) -> Connector_PinHeader_2.00mm:PinHeader_1x02_P2.00mm_Vertical
- J19: footprint Connector_PinHeader_1.00mm:PinHeader_1x02_P1.00mm_Vertical_SMD_Pin1Right -> Connector_PinHeader_2.00mm:PinHeader_1x02_P2.00mm_Vertical
- Q5: footprint Package_TO_SOT_THT:TO-92_Inline -> OldComp:Transistor_TO92_EBC_254
Changed lines of the file:
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@@
 			)
 		)
-		(property "Footprint" ""
+		(property "Footprint" "Capacitor_THT:C_Axial_L3.8mm_D2.6mm_P10.00mm_Horizontal"
 			(at 119.38 59.69 0)
 			(effects
@@
 			)
 		)
-		(property "Footprint" ""
+		(property "Footprint" "Capacitor_THT:C_Axial_L3.8mm_D2.6mm_P10.00mm_Horizontal"
 			(at 149.86 128.27 0)
 			(effects
@@
 			)
 		)
-		(property "Footprint" ""
+		(property "Footprint" "Capacitor_THT:C_Axial_L3.8mm_D2.6mm_P10.00mm_Horizontal"
 			(at 138.43 128.27 0)
 			(effects
@@
 			)
 		)
-		(property "Footprint" ""
+		(property "Footprint" "Capacitor_THT:C_Axial_L3.8mm_D2.6mm_P10.00mm_Horizontal"
 			(at 115.57 128.27 0)
 			(effects
@@
 			)
 		)
-		(property "Footprint" ""
+		(property "Footprint" "Capacitor_THT:C_Axial_L3.8mm_D2.6mm_P10.00mm_Horizontal"
 			(at 127 128.27 0)
 			(effects
@@
 			)
 		)
-		(property "Footprint" ""
+		(property "Footprint" "OldComp:Cap_Cer_762"
 			(at 166.37 142.24 0)
 			(effects
@@
 			)
 		)
-		(property "Footprint" ""
+		(property "Footprint" "Capacitor_THT:C_Axial_L3.8mm_D2.6mm_P10.00mm_Horizontal"
 			(at 154.94 254 0)
 			(effects
@@
 			)
 		)
-		(property "Footprint" ""
+		(property "Footprint" "Capacitor_THT:C_Disc_D5.0mm_W2.5mm_P2.50mm"
 			(at 167.64 226.06 0)
 			(effects
@@
 			)
 		)
-		(property "Footprint" "Connector_PinHeader_1.00mm:PinHeader_1x02_P1.00mm_Vertical_SMD_Pin1Right"
+		(property "Footprint" "Connector_PinHeader_2.00mm:PinHeader_1x02_P2.00mm_Vertical"
 			(at 214.63 161.29 0)
 			(effects
@@
 			)
 		)
-		(property "Footprint" ""
+		(property "Footprint" "Capacitor_THT:C_Axial_L3.8mm_D2.6mm_P10.00mm_Horizontal"
 			(at 247.65 220.98 0)
 			(effects
@@
 			)
 		)
-		(property "Footprint" ""
+		(property "Footprint" "Capacitor_THT:C_Axial_L3.8mm_D2.6mm_P10.00mm_Horizontal"
 			(at 284.48 218.44 0)
 			(effects
@@
 			)
 		)
-		(property "Footprint" ""
+		(property "Footprint" "Connector_PinHeader_2.00mm:PinHeader_1x02_P2.00mm_Vertical"
 			(at 300.99 203.2 0)
 			(effects
@@
 			)
 		)
-		(property "Footprint" "Package_TO_SOT_THT:TO-92_Inline"
+		(property "Footprint" "OldComp:Transistor_TO92_EBC_254"
 			(at 274.32 218.44 0)
 			(effects
@@
 		(dnp no)
 		(property "Reference" "UC5"
-			(at 245.11 22.4282 0)
+			(at 245.11 30.226 0)
 			(effects
 				(font
@@
 		(dnp no)
 		(property "Reference" "UB8"
-			(at 252.73 123.825 0)
+			(at 253.238 132.08 0)
 			(effects
 				(font
@@
 		)
 		(property "Value" "S02"
-			(at 252.73 126.1364 0)
+			(at 252.73 126.746 0)
 			(effects
 				(font

Commit message: add change apple2e-3
Parts:
- removed SA1: SoundAmp, Ferrite_THT:LairdTech_28C0236-0JW-10, symbol Apple_IIe_Symbols:SoundAmp
- C36: footprint OldComp:Cap_Cer_762 -> Capacitor_THT:C_Axial_L3.8mm_D2.6mm_P10.00mm_Horizontal
- C79: value .1uF -> 1uF; footprint Capacitor_THT:C_Axial_L3.8mm_D2.6mm_P10.00mm_Horizontal -> PCM_Capacitor_THT_AKL:CP_Axial_L10.0mm_D6.0mm_P15.00mm_Horizontal
- CR2: footprint (none) -> LED_THT:LED_D5.0mm_Clear
- CR4: footprint (none) -> Diode_THT:D_A-405_P12.70mm_Horizontal
- Q5: footprint OldComp:Transistor_TO92_EBC_254 -> Package_TO_SOT_THT:TO-18-3; symbol Device:Q_NPN_Darlington_EBC -> Transistor_BJT:BC107
- X2: footprint Jumper:SolderJumper-2_P1.3mm_Open_RoundedPad1.0x1.5mm -> Jumper:SolderJumper-2_P1.3mm_Bridged2Bar_RoundedPad1.0x1.5mm
