File: POWER_CONNECTORS-4.kicad_sch (KiCad schematic)
At the start: 41 parts, among them J0 Conn_02x30_Counter_Clockwise, J1 Conn_02x25_Counter_Clockwise, J14 Conn_01x06, J15 Conn_02x08_Counter_Clockwise, J16 Conn_01x11, J17 Conn_02x13_Odd_Even, J2 Conn_02x25_Counter_Clockwise, J20 Conn_01x04, J3 Conn_02x25_Counter_Clockwise, J4 Conn_02x25_Counter_Clockwise, J5 Conn_02x25_Counter_Clockwise, J6 Conn_02x25_Counter_Clockwise, J7 Conn_02x25_Counter_Clockwise, J8 DB9_Female, U8 S02, X7 SolderJumper_2_Open

Commit message: add change apple2e
Parts:
- removed U8: S02, Package_DIP:DIP-14_W7.62mm_Socket_LongPads, symbol 74xx:7402
- J1: footprint PCM_MA_Connector_AppleII:EDAC_395-050-520-201_CounterClockwise -> Package_DIP:DIP-16_W7.62mm_Socket_LongPads
- J8: footprint (none) -> Connector_Dsub:DSUB-9_Socket_Horizontal_P2.77x2.84mm_EdgePinOffset7.70mm_Housed_MountingHolesOffset9.12mm
- UB8, UC5, UE1: footprint (none) -> Package_DIP:DIP-14_W7.62mm_Socket_LongPads
- UC1: footprint (none) -> Package_DIP:DIP-16_W7.62mm_Socket_LongPads
- X7: footprint (none) -> Jumper:SolderJumper-2_P1.3mm_Open_RoundedPad1.0x1.5mm

Commit message: add change apple2e-2
Parts:
- C1-7,10: footprint Capacitor_THT:C_Disc_D3.4mm_W2.1mm_P2.50mm -> Capacitor_THT:C_Axial_L3.8mm_D2.6mm_P10.00mm_Horizontal
- C12, C15, C53,54,72,82: footprint (none) -> PCM_Capacitor_THT_AKL:CP_Axial_L10.0mm_D6.0mm_P15.00mm_Horizontal
- C13, C16,19-24, C18, C26-31,33, C38,39,48-52,55-59,61-69,73-76,78,81,84-89, C41-47, C60: footprint (none) -> Capacitor_THT:C_Axial_L3.8mm_D2.6mm_P10.00mm_Horizontal
- C17: footprint (none) -> PCM_Capacitor_THT_AKL:CP_Axial_L10.0mm_D6.0mm_P15.00mm_Horizontal; symbol Device:C_Polarized_Small -> PCM_Capacitor_AKL:CP_Axial_L10.0mm_D6.0mm_P15.00mm
- C8,9: footprint Capacitor_THT:C_Radial_D5.0mm_H11.0mm_P2.00mm -> PCM_Capacitor_THT_AKL:CP_Axial_L10.0mm_D6.0mm_P15.00mm_Horizontal
- J14: footprint (none) -> OldComp:Conn_Power_AT_6pin
- J15: footprint (none) -> Package_DIP:DIP-16_W10.16mm_LongPads
- J20: footprint (none) -> Connector_PinHeader_1.00mm:PinHeader_1x04_P1.00mm_Vertical
- L1, L2, L4, L5, L6: footprint (none) -> Inductor_THT:L_Radial_D6.0mm_P4.00mm
Other:
- moved on the sheet: C17
Changed lines of the file:
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@@
 	(wire
 		(pts
-			(xy 242.57 143.51) (xy 242.57 144.78)
-		)
-		(stroke
-			(width 0)
-			(type default)
-		)
-	)
-	(wire
-		(pts
 			(xy 280.035 220.98) (xy 283.21 220.98)
 		)
@@
 			)
 		)
-		(property "Footprint" ""
+		(property "Footprint" "Connector_PinHeader_1.00mm:PinHeader_1x04_P1.00mm_Vertical"
 			(at 100.33 147.32 0)
 			(effects
@@
 			)
 		)
-		(property "Footprint" ""
+		(property "Footprint" "Package_DIP:DIP-16_W10.16mm_LongPads"
 			(at 358.775 169.545 0)
 			(effects
@@
 			)
 		)
-		(property "Footprint" ""
+		(property "Footprint" "OldComp:Conn_Power_AT_6pin"
 			(at 219.71 144.78 0)
 			(effects
@@
 	)
 	(symbol
-		(lib_id "Device:C_Polarized_Small")
-		(at 242.57 140.97 180)
+		(lib_id "PCM_Capacitor_AKL:CP_Axial_L10.0mm_D6.0mm_P15.00mm")
+		(at 242.57 142.24 180)
 		(unit 1)
 		(exclude_from_sim no)
@@
 		(dnp no)
 		(property "Reference" "C17"
-			(at 244.8052 139.8016 0)
+			(at 244.8052 141.0716 0)
 			(effects
 				(font
@@
 		)
 		(property "Value" "10uF 6V"
-			(at 244.8052 142.113 0)
+			(at 244.8052 143.383 0)
 			(effects
 				(font
@@
 			)
 		)
-		(property "Footprint" ""
-			(at 242.57 140.97 0)
+		(property "Footprint" "PCM_Capacitor_THT_AKL:CP_Axial_L10.0mm_D6.0mm_P15.00mm_Horizontal"
+			(at 242.57 132.08 0)
 			(effects
 				(font
@@
 		)
 		(property "Datasheet" "~"
-			(at 242.57 140.97 0)
+			(at 242.57 142.24 0)
 			(effects
 				(font
@@
 			)
 		)
-		(property "Description" "Polarized capacitor, small symbol"
-			(at 242.57 140.97 0)
+		(property "Description" "THT Axial Electrolytic Capacitor, 10.0mm Length, 6.0mm Diameter, 15.00mm Pitch, European Symbol, Alternate KiCad Library"
+			(at 242.57 142.24 0)
 			(effects
 				(font
@@
 	(symbol
 		(lib_id "power:GND")
-		(at 242.57 144.78 0)
+		(at 242.57 146.05 0)
 		(unit 1)
 		(exclude_from_sim no)
@@
 		(dnp no)
 		(property "Reference" "#PWR0100"
-			(at 242.57 151.13 0)
+			(at 242.57 152.4 0)
 			(effects
 				(font
@@
 		)
 		(property "Value" "GND"
-			(at 242.697 149.1742 0)
+			(at 242.697 150.4442 0)
 			(effects
 				(font
@@
 		)
 		(property "Footprint" ""
-			(at 242.57 144.78 0)
+			(at 242.57 146.05 0)
 			(effects
 				(font
@@
 		)
 		(property "Datasheet" ""
-			(at 242.57 144.78 0)
+			(at 242.57 146.05 0)
 			(effects
 				(font
@@
 		)
 		(property "Description" "Power symbol creates a global label with name \"GND\" , ground"
-			(at 242.57 144.78 0)
+			(at 242.57 146.05 0)
 			(effects
 				(font
@@
 			)
 		)
-		(property "Footprint" ""
+		(property "Footprint" "Capacitor_THT:C_Axial_L3.8mm_D2.6mm_P10.00mm_Horizontal"
 			(at 256.54 140.97 0)
 			(effects
@@
 			)
 		)
-		(property "Footprint" ""
+		(property "Footprint" "Inductor_THT:L_Radial_D6.0mm_P4.00mm"
 			(at 261.62 137.16 0)
 			(effects
@@
 			)
 		)
-		(property "Footprint" ""
+		(property "Footprint" "Capacitor_THT:C_Axial_L3.8mm_D2.6mm_P10.00mm_Horizontal"
 			(at 280.67 140.97 0)
 			(effects
@@
 			)
 		)
-		(property "Footprint" ""
+		(property "Footprint" "Inductor_THT:L_Radial_D6.0mm_P4.00mm"
 			(at 261.62 156.21 0)
 			(effects
@@
 			)
 		)
-		(property "Footprint" ""
+		(property "Footprint" "PCM_Capacitor_THT_AKL:CP_Axial_L10.0mm_D6.0mm_P15.00mm_Horizontal"
 			(at 266.7 160.02 0)
 			(effects
@@
 			)
 		)
-		(property "Footprint" ""
+		(property "Footprint" "Capacitor_THT:C_Axial_L3.8mm_D2.6mm_P10.00mm_Horizontal"
 			(at 280.67 160.02 0)
 			(effects
@@
 			)
 		)
-		(property "Footprint" ""
+		(property "Footprint" "Capacitor_THT:C_Axial_L3.8mm_D2.6mm_P10.00mm_Horizontal"
 			(at 280.67 175.895 0)
 			(effects
@@
 			)
 		)
-		(property "Footprint" ""
+		(property "Footprint" "PCM_Capacitor_THT_AKL:CP_Axial_L10.0mm_D6.0mm_P15.00mm_Horizontal"
 			(at 234.95 193.675 0)
 			(effects
@@
 			)
 		)
-		(property "Footprint" ""
+		(property "Footprint" "Capacitor_THT:C_Axial_L3.8mm_D2.6mm_P10.00mm_Horizontal"
 			(at 248.92 193.675 0)
 			(effects
@@
 			)
 		)
-		(property "Footprint" ""
+		(property "Footprint" "Inductor_THT:L_Radial_D6.0mm_P4.00mm"
 			(at 267.335 189.865 0)
 			(effects
@@
 			)
 		)
-		(property "Footprint" ""
+		(property "Footprint" "Capacitor_THT:C_Axial_L3.8mm_D2.6mm_P10.00mm_Horizontal"
 			(at 280.67 193.675 0)
 			(effects
@@
 			)
 		)
-		(property "Footprint" ""
+		(property "Footprint" "Inductor_THT:L_Radial_D6.0mm_P4.00mm"
 			(at 243.84 220.98 0)
 			(effects
@@
 			)
 		)
-		(property "Footprint" "Capacitor_THT:C_Radial_D5.0mm_H11.0mm_P2.00mm"
+		(property "Footprint" "PCM_Capacitor_THT_AKL:CP_Axial_L10.0mm_D6.0mm_P15.00mm_Horizontal"
 			(at 262.255 224.79 0)
 			(effects
@@
 			)
 		)
-		(property "Footprint" "Capacitor_THT:C_Disc_D3.4mm_W2.1mm_P2.50mm"
+		(property "Footprint" "Capacitor_THT:C_Axial_L3.8mm_D2.6mm_P10.00mm_Horizontal"
 			(at 280.035 224.79 0)
 			(effects
@@
 			)
 		)
-		(property "Footprint" ""
+		(property "Footprint" "Inductor_THT:L_Radial_D6.0mm_P4.00mm"
 			(at 243.84 243.205 0)
 			(effects
@@
 			)
 		)
-		(property "Footprint" ""
+		(property "Footprint" "PCM_Capacitor_THT_AKL:CP_Axial_L10.0mm_D6.0mm_P15.00mm_Horizontal"
 			(at 262.89 247.015 0)
 			(effects
@@
 			)
 		)
-		(property "Footprint" ""
+		(property "Footprint" "Capacitor_THT:C_Axial_L3.8mm_D2.6mm_P10.00mm_Horizontal"
 			(at 280.67 247.015 0)
 			(effects

Commit message: add change apple2e-3
Parts:
- removed J1: Conn_02x25_Counter_Clockwise, Package_DIP:DIP-16_W7.62mm_Socket_LongPads, symbol Connector_Generic:Conn_02x25_Counter_Clockwise
- removed J2, J3, J4, J5, J6, J7: Conn_02x25_Counter_Clockwise, PCM_MA_Connector_AppleII:EDAC_395-050-520-201_CounterClockwise, symbol Connector_Generic:Conn_02x25_Counter_Clockwise
- added J1, J2, J3, J4, J5, J6, J7: Bus_Apple_II_Computer_Side, PCM_MA_Connector_AppleII:EDAC_395-050-520-201_CounterClockwise, symbol PCM_MA_Connector_AppleII:Bus_Apple_II_Computer_Side
- CR1: footprint (none) -> LED_THT:LED_D5.0mm_Clear; symbol Device:LED_Small -> PCM_SL_Devices:LED
- J0: footprint (none) -> PCM_MA_Connector_AppleII:EDAC_395-060-520-201_CounterClockwise
- J16: footprint (none) -> Connector_PinHeader_1.00mm:PinHeader_1x11_P1.00mm_Vertical
- J17: footprint (none) -> Connector_IDC:IDC-Header_2x13_P2.54mm_Vertical
Connections:
- net +12C: now also J1.50 (+12V), J2.50 (+12V), J3.50 (+12V), J4.50 (+12V), J5.50 (+12V), J6.50 (+12V), J7.50 (+12V)
- net +12V: now also CR1.1; no longer CR1.2 (A)
- net +5C: now also J1.25 (+5V), J2.25 (+5V), J3.25 (+5V), J4.25 (+5V), J5.25 (+5V), J6.25 (+5V), J7.25 (+5V)
- net -12C: now also J1.33 (-12V), J2.33 (-12V), J3.33 (-12V), J4.33 (-12V), J5.33 (-12V), J6.33 (-12V), J7.33 (-12V)
- net -5C: now also J1.34 (-5V), J2.34 (-5V), J3.34 (-5V), J4.34 (-5V), J5.34 (-5V), J6.34 (-5V), J7.34 (-5V)
- net 3.58M: now also J7.35 (TESTPIN)
- net 7M: now also J1.36 (7M), J2.36 (7M), J3.36 (7M), J4.36 (7M), J5.36 (7M), J6.36 (7M), J7.36 (7M)
- net A0: now also J1.2 (A0), J2.2 (A0), J3.2 (A0), J4.2 (A0), J5.2 (A0), J6.2 (A0), J7.2 (A0)
- net A1: now also J1.3 (A1), J2.3 (A1), J3.3 (A1), J4.3 (A1), J5.3 (A1), J6.3 (A1), J7.3 (A1)
- net A10: now also J1.12 (A10), J2.12 (A10), J3.12 (A10), J4.12 (A10), J5.12 (A10), J6.12 (A10), J7.12 (A10)
- net A11: now also J1.13 (A11), J2.13 (A11), J3.13 (A11), J4.13 (A11), J5.13 (A11), J6.13 (A11), J7.13 (A11)
- net A12: now also J1.14 (A12), J2.14 (A12), J3.14 (A12), J4.14 (A12), J5.14 (A12), J6.14 (A12), J7.14 (A12)
- net A13: now also J1.15 (A13), J2.15 (A13), J3.15 (A13), J4.15 (A13), J5.15 (A13), J6.15 (A13), J7.15 (A13)
- net A14: now also J1.16 (A14), J2.16 (A14), J3.16 (A14), J4.16 (A14), J5.16 (A14), J6.16 (A14), J7.16 (A14)
- net A15: now also J1.17 (A15), J2.17 (A15), J3.17 (A15), J4.17 (A15), J5.17 (A15), J6.17 (A15), J7.17 (A15)
- net A2: now also J1.4 (A2), J2.4 (A2), J3.4 (A2), J4.4 (A2), J5.4 (A2), J6.4 (A2), J7.4 (A2)
- net A3: now also J1.5 (A3), J2.5 (A3), J3.5 (A3), J4.5 (A3), J5.5 (A3), J6.5 (A3), J7.5 (A3)
- net A4: now also J1.6 (A4), J2.6 (A4), J3.6 (A4), J4.6 (A4), J5.6 (A4), J6.6 (A4), J7.6 (A4)
- net A5: now also J1.7 (A5), J2.7 (A5), J3.7 (A5), J4.7 (A5), J5.7 (A5), J6.7 (A5), J7.7 (A5)
- net A6: now also J1.8 (A6), J2.8 (A6), J3.8 (A6), J4.8 (A6), J5.8 (A6), J6.8 (A6), J7.8 (A6)
- net A7: now also J1.9 (A7), J2.9 (A7), J3.9 (A7), J4.9 (A7), J5.9 (A7), J6.9 (A7), J7.9 (A7)
- net A8: now also J1.10 (A8), J2.10 (A8), J3.10 (A8), J4.10 (A8), J5.10 (A8), J6.10 (A8), J7.10 (A8)
- net A9: now also J1.11 (A9), J2.11 (A9), J3.11 (A9), J4.11 (A9), J5.11 (A9), J6.11 (A9), J7.11 (A9)
- net D0: now also J1.49 (D0), J2.49 (D0), J3.49 (D0), J4.49 (D0), J5.49 (D0), J6.49 (D0), J7.49 (D0)
- net D1: now also J1.48 (D1), J2.48 (D1), J3.48 (D1), J4.48 (D1), J5.48 (D1), J6.48 (D1), J7.48 (D1)
- net D2: now also J1.47 (D2), J2.47 (D2), J3.47 (D2), J4.47 (D2), J5.47 (D2), J6.47 (D2), J7.47 (D2)
- net D3: now also J1.46 (D3), J2.46 (D3), J3.46 (D3), J4.46 (D3), J5.46 (D3), J6.46 (D3), J7.46 (D3)
- net D4: now also J1.45 (D4), J2.45 (D4), J3.45 (D4), J4.45 (D4), J5.45 (D4), J6.45 (D4), J7.45 (D4)
- net D5: now also J1.44 (D5), J2.44 (D5), J3.44 (D5), J4.44 (D5), J5.44 (D5), J6.44 (D5), J7.44 (D5)
- net D6: now also J1.43 (D6), J2.43 (D6), J3.43 (D6), J4.43 (D6), J5.43 (D6), J6.43 (D6), J7.43 (D6)
- net D7: now also J1.42 (D7), J2.42 (D7), J3.42 (D7), J4.42 (D7), J5.42 (D7), J6.42 (D7), J7.42 (D7)
- net DMA1: now also J1.24 (DMA_OUT), J2.27 (DMA_IN)
- net DMA2: now also J2.24 (DMA_OUT), J3.27 (DMA_IN)
- net DMA3: now also J3.24 (DMA_OUT), J4.27 (DMA_IN)
- net DMA4: now also J4.24 (DMA_OUT), J5.27 (DMA_IN)
- net DMA5: now also J5.24 (DMA_OUT), J6.27 (DMA_IN)
- net DMA6: now also J6.24 (DMA_OUT), J7.27 (DMA_IN)
- net GND: now also J1.26 (GND), J2.26 (GND), J3.26 (GND), J4.26 (GND), J5.26 (GND), J6.26 (GND), J7.26 (GND)
- net INT1: now also J1.23 (INT_OUT), J2.28 (INT_IN)
- net INT2: now also J2.23 (INT_OUT), J3.28 (INT_IN)
- net INT3: now also J3.23 (INT_OUT), J4.28 (INT_IN)
- net INT4: now also J4.23 (INT_OUT), J5.28 (INT_IN)
- net INT5: now also J5.23 (INT_OUT), J6.28 (INT_IN)
- net INT6: now also J6.23 (INT_OUT), J7.28 (INT_IN)
- net PH0: now also J1.40 (Φ0), J2.40 (Φ0), J3.40 (Φ0), J4.40 (Φ0), J5.40 (Φ0), J6.40 (Φ0), J7.40 (Φ0)
- net PH1: now also J1.38 (Φ1), J2.38 (Φ1), J3.38 (Φ1), J4.38 (Φ1), J5.38 (Φ1), J6.38 (Φ1), J7.38 (Φ1)
- net Q3: now also J1.37 (Q3), J2.37 (Q3), J3.37 (Q3), J4.37 (Q3), J5.37 (Q3), J6.37 (Q3), J7.37 (Q3)
- net RDY: now also J1.21 (RDY), J2.21 (RDY), J3.21 (RDY), J4.21 (RDY), J5.21 (RDY), J6.21 (RDY), J7.21 (RDY)
- net R_~{W}: now also J1.18 (R/~{W}), J2.18 (R/~{W}), J3.18 (R/~{W}), J4.18 (R/~{W}), J5.18 (R/~{W}), J6.18 (R/~{W}), J7.18 (R/~{W})
- net UPSYNC: now also J1.39 (USER1), J2.39 (USER1), J3.39 (USER1), J4.39 (USER1), J5.39 (USER1), J6.39 (USER1), J7.39 (USER1)
- net ~{CLKEN}: now also J3.19 (TESTPIN)
- net ~{DEV1}: now also J1.41 (~{DEVICE_SELECT})
- net ~{DEV2}: now also J2.41 (~{DEVICE_SELECT})
- net ~{DEV3}: now also J3.41 (~{DEVICE_SELECT})
- net ~{DEV4}: now also J4.41 (~{DEVICE_SELECT})
- net ~{DEV5}: now also J5.41 (~{DEVICE_SELECT})
- net ~{DEV6}: now also J6.41 (~{DEVICE_SELECT})
- net ~{DEV7}: now also J7.41 (~{DEVICE_SELECT})
- net ~{DMA}: now also J1.22 (~{DMA}), J2.22 (~{DMA}), J3.22 (~{DMA}), J4.22 (~{DMA}), J5.22 (~{DMA}), J6.22 (~{DMA}), J7.22 (~{DMA})
- net ~{ENKBD}: now also J3.35 (TESTPIN)
- net ~{INH}: now also J1.32 (~{INH}), J2.32 (~{INH}), J3.32 (~{INH}), J4.32 (~{INH}), J5.32 (~{INH}), J6.32 (~{INH}), J7.32 (~{INH})
- net ~{IOSEL1}: now also J1.1 (~{I/O_SELECT})
- net ~{IOSEL2}: now also J2.1 (~{I/O_SELECT})
- net ~{IOSEL3}: now also J3.1 (~{I/O_SELECT})
- net ~{IOSEL4}: now also J4.1 (~{I/O_SELECT})
- net ~{IOSEL5}: now also J5.1 (~{I/O_SELECT})
- net ~{IOSEL6}: now also J6.1 (~{I/O_SELECT})
- net ~{IOSEL7}: now also J7.1 (~{I/O_SELECT})
- net ~{IOSTRB}: now also J1.20 (~{I/O_STROBE}), J2.20 (~{I/O_STROBE}), J3.20 (~{I/O_STROBE}), J4.20 (~{I/O_STROBE}), J5.20 (~{I/O_STROBE}), J6.20 (~{I/O_STROBE}), J7.20 (~{I/O_STROBE})
- net ~{IRQ}: now also J1.30 (~{IRQ}), J2.30 (~{IRQ}), J3.30 (~{IRQ}), J4.30 (~{IRQ}), J5.30 (~{IRQ}), J6.30 (~{IRQ}), J7.30 (~{IRQ})
- net ~{NMI}: now also J1.29 (~{NMI}), J2.29 (~{NMI}), J3.29 (~{NMI}), J4.29 (~{NMI}), J5.29 (~{NMI}), J6.29 (~{NMI}), J7.29 (~{NMI})
- net ~{RESET}: now also J1.31 (~{RES}), J2.31 (~{RES}), J3.31 (~{RES}), J4.31 (~{RES}), J5.31 (~{RES}), J6.31 (~{RES}), J7.31 (~{RES})
- net ~{SYNC}: now also J7.19 (TESTPIN)
- net INT7: now reaches X7.1 (A)
- net INT7: now also J7.23 (INT_OUT)
- net at R1.1: now also CR1.2; no longer CR1.1 (K)
Other:
- moved on the sheet: X7
