File: TIMING_VIDEO-3.kicad_sch (KiCad schematic)
At the start: 59 parts, among them J10 CASSETTE OUT, J11 NTSC OUT, J12 Conn_01x01, J13 Conn_01x04, Q1 2N3906, Q2 2N3904, Q4 2N4258, Q6 2N4258, X3 SolderJumper_2_Open, Y1 Crystal_Small

Commit message: add change apple2e
Parts:
- J10: footprint (none) -> Connector_Audio:Jack_3.5mm_CUI_SJ1-3525N_Horizontal
- J11: footprint (none) -> Connector_Coaxial:BNC_Win_364A2x95_Horizontal
- Q4, Q6: footprint (none) -> Package_TO_SOT_THT:TO-92_Inline
- RP1: footprint Resistor_THT:R_Array_SIP10 -> Resistor_THT:R_Array_SIP9
- UB8, UC5, UE1: footprint (none) -> Package_DIP:DIP-14_W7.62mm_Socket_LongPads
- UC1, UF5: footprint (none) -> Package_DIP:DIP-16_W7.62mm_Socket_LongPads
- UD1: footprint (none) -> Package_DIP:DIP-20_W7.62mm_LongPads
- UD3: footprint (none) -> Package_DIP:DIP-20_W7.62mm_Socket_LongPads
- UF4: footprint (none) -> Package_DIP:DIP-24_18.0mmx34.29mm_W15.24mm_Socket_LongPads
- VA1: footprint (none) -> Package_DIP:DIP-40_W15.24mm_Socket_LongPads
- X3: footprint (none) -> Jumper:SolderJumper-2_P1.3mm_Open_RoundedPad1.0x1.5mm
Connections:
- net +5V: now also UD1.20 (VCC), UD3.20 (VCC), UF5.16 (VCC)
- net GND: now also UD1.10 (GND), UD3.10 (GND), UF5.8 (GND)

Commit message: add change apple2e-2
Parts:
- C25, C32, C90, C91, C92, C93: footprint (none) -> Capacitor_THT:C_Disc_D5.0mm_W2.5mm_P2.50mm
- C77, C83: footprint (none) -> Capacitor_THT:C_Axial_L3.8mm_D2.6mm_P10.00mm_Horizontal
- J12: footprint (none) -> Connector_PinHeader_1.00mm:PinHeader_1x01_P1.00mm_Vertical
- J13: footprint (none) -> Connector_PinHeader_1.00mm:PinHeader_1x04_P1.00mm_Vertical
- L3: footprint (none) -> Inductor_THT:L_Radial_D6.0mm_P4.00mm
- Q4, Q6: symbol Device:Q_PNP_EBC -> Transistor_BJT:2N3904
Changed lines of the file:
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@@
 		(dnp no)
 		(property "Reference" "UF5"
-			(at 257.556 56.642 0)
+			(at 260.35 71.628 0)
 			(effects
 				(font
@@
 		)
 		(property "Value" "LS166"
-			(at 258.064 59.182 0)
+			(at 260.35 75.438 0)
 			(effects
 				(font
@@
 		(dnp no)
 		(property "Reference" "UC5"
-			(at 288.29 42.7482 0)
+			(at 288.036 50.8 0)
 			(effects
 				(font
@@
 		(dnp no)
 		(property "Reference" "UB8"
-			(at 288.29 71.755 0)
+			(at 288.798 80.01 0)
 			(effects
 				(font
@@
 	)
 	(symbol
-		(lib_id "Device:Q_PNP_EBC")
+		(lib_id "Transistor_BJT:2N3904")
 		(at 59.69 196.85 0)
 		(mirror x)
@@
 		)
 		(property "Footprint" "Package_TO_SOT_THT:TO-92_Inline"
-			(at 64.77 199.39 0)
+			(at 64.77 194.945 0)
 			(effects
 				(font
 					(size 1.27 1.27)
+					(italic yes)
 				)
+				(justify left)
 				(hide yes)
 			)
 		)
-		(property "Datasheet" "~"
+		(property "Datasheet" "https://www.onsemi.com/pub/Collateral/2N3903-D.PDF"
 			(at 59.69 196.85 0)
 			(effects
@@
 					(size 1.27 1.27)
 				)
+				(justify left)
 				(hide yes)
 			)
 		)
-		(property "Description" ""
+		(property "Description" "0.2A Ic, 40V Vce, Small Signal NPN Transistor, TO-92"
 			(at 59.69 196.85 0)
 			(effects
@@
 					(size 1.27 1.27)
 				)
+				(hide yes)
+			)
+		)
+		(property "Sim.Device" "NPN"
+			(at 59.69 196.85 0)
+			(effects
+				(font
+					(size 1.27 1.27)
+				)
+				(hide yes)
+			)
+		)
+		(property "Sim.Pins" "1=E 2=B 3=C"
+			(at 59.69 196.85 0)
+			(effects
+				(font
+					(size 1.27 1.27)
+				)
+				(hide yes)
 			)
 		)
@@
 	)
 	(symbol
-		(lib_id "Device:Q_PNP_EBC")
+		(lib_id "Transistor_BJT:2N3904")
 		(at 80.01 196.85 180)
 		(unit 1)
@@
 		)
 		(property "Footprint" "Package_TO_SOT_THT:TO-92_Inline"
-			(at 74.93 199.39 0)
+			(at 74.93 194.945 0)
 			(effects
 				(font
 					(size 1.27 1.27)
+					(italic yes)
 				)
+				(justify left)
 				(hide yes)
 			)
 		)
-		(property "Datasheet" "~"
+		(property "Datasheet" "https://www.onsemi.com/pub/Collateral/2N3903-D.PDF"
 			(at 80.01 196.85 0)
 			(effects
@@
 					(size 1.27 1.27)
 				)
+				(justify left)
 				(hide yes)
 			)
 		)
-		(property "Description" ""
+		(property "Description" "0.2A Ic, 40V Vce, Small Signal NPN Transistor, TO-92"
+			(at 80.01 196.85 0)
+			(effects
+				(font
+					(size 1.27 1.27)
+				)
+				(hide yes)
+			)
+		)
+		(property "Sim.Device" "NPN"
+			(at 80.01 196.85 0)
+			(effects
+				(font
+					(size 1.27 1.27)
+				)
+				(hide yes)
+			)
+		)
+		(property "Sim.Pins" "1=E 2=B 3=C"
 			(at 80.01 196.85 0)
 			(effects
@@
 					(size 1.27 1.27)
 				)
+				(hide yes)
 			)
 		)
@@
 		(dnp no)
 		(property "Reference" "UE1"
-			(at 100.33 200.2282 0)
+			(at 99.568 208.28 0)
 			(effects
 				(font
@@
 		)
 		(property "Value" "LS125"
-			(at 100.33 202.5396 0)
+			(at 101.092 203.708 0)
 			(effects
 				(font
@@
 		(dnp no)
 		(property "Reference" "UC5"
-			(at 113.03 149.225 0)
+			(at 112.776 157.48 0)
 			(effects
 				(font
@@
 		)
 		(property "Value" "LS10"
-			(at 113.03 151.5364 0)
+			(at 112.014 151.638 0)
 			(effects
 				(font
@@
 			)
 		)
-		(property "Footprint" ""
+		(property "Footprint" "Capacitor_THT:C_Axial_L3.8mm_D2.6mm_P10.00mm_Horizontal"
 			(at 96.52 185.42 0)
 			(effects
@@
 			)
 		)
-		(property "Footprint" ""
+		(property "Footprint" "Capacitor_THT:C_Axial_L3.8mm_D2.6mm_P10.00mm_Horizontal"
 			(at 26.67 214.63 0)
 			(effects
@@
 			)
 		)
-		(property "Footprint" ""
+		(property "Footprint" "Capacitor_THT:C_Disc_D5.0mm_W2.5mm_P2.50mm"
 			(at 288.29 226.06 0)
 			(effects
@@
 			)
 		)
-		(property "Footprint" ""
+		(property "Footprint" "Capacitor_THT:C_Disc_D5.0mm_W2.5mm_P2.50mm"
 			(at 298.45 226.06 0)
 			(effects
@@
 			)
 		)
-		(property "Footprint" ""
+		(property "Footprint" "Capacitor_THT:C_Disc_D5.0mm_W2.5mm_P2.50mm"
 			(at 309.88 226.06 0)
 			(effects
@@
 			)
 		)
-		(property "Footprint" ""
+		(property "Footprint" "Capacitor_THT:C_Disc_D5.0mm_W2.5mm_P2.50mm"
 			(at 304.8 87.63 0)
 			(effects
@@
 			)
 		)
-		(property "Footprint" ""
+		(property "Footprint" "Inductor_THT:L_Radial_D6.0mm_P4.00mm"
 			(at 314.96 87.63 0)
 			(effects
@@
 			)
 		)
-		(property "Footprint" ""
+		(property "Footprint" "Capacitor_THT:C_Disc_D5.0mm_W2.5mm_P2.50mm"
 			(at 330.2 88.9 0)
 			(effects
@@
 			)
 		)
-		(property "Footprint" ""
+		(property "Footprint" "Connector_PinHeader_1.00mm:PinHeader_1x04_P1.00mm_Vertical"
 			(at 372.11 91.44 0)
 			(effects
@@
 			)
 		)
-		(property "Footprint" ""
+		(property "Footprint" "Connector_PinHeader_1.00mm:PinHeader_1x01_P1.00mm_Vertical"
 			(at 377.19 83.82 0)
 			(effects
@@
 			)
 		)
-		(property "Footprint" ""
+		(property "Footprint" "Capacitor_THT:C_Disc_D5.0mm_W2.5mm_P2.50mm"
 			(at 332.74 238.76 0)
 			(effects

Commit message: add change apple2e-3
Parts:
- removed C77: .01uF, Capacitor_THT:C_Axial_L3.8mm_D2.6mm_P10.00mm_Horizontal, symbol Device:C_Small
- removed J10: CASSETTE OUT, Connector_Audio:Jack_3.5mm_CUI_SJ1-3525N_Horizontal, symbol Connector:Conn_Coaxial
- removed NT1: NetTie_2, symbol Device:NetTie_2
- removed OSC1, OSC2: Oscillator, symbol Apple_IIe_Symbols:Oscillator
- removed R33: 10R, Resistor_THT:R_Axial_DIN0204_L3.6mm_D1.6mm_P7.62mm_Horizontal, symbol Device:R_Small
- removed VA1: VideoAmp, Package_DIP:DIP-40_W15.24mm_Socket_LongPads, symbol Apple_IIe_Symbols:VideoAmp
- added J10: AUDIO OUT, Connector_Audio:Jack_3.5mm_CUI_SJ1-3525N_Horizontal, symbol Connector_Audio:AudioJack3_Ground
Connections:
- net GND: now also J10.G
- net at R6.1, R9.2: now also J10.T
- no-connect marks 2 -> 4
